File: kicad/patamana.kicad_pcb (KiCad board)
At the start: 2 copper layers, 30.5 x 69.8 mm, 59 parts, among them J1 TRRSJack, J2 TRRSJack, J3 Conn_01x02, SW1 SW_Push, SW2 SW_Push, SW3 SW_DPDT_x2, SW4 SW_DPDT_x2, U1 XIAO_ESP32S3, U2 74HC165, U3 OLED(I2C), U4 74HC165, U5 74HC165, U6 74HC165

Commit message: 整理:名前の整理
Parts:
- C1, C2, C3, C4, C5, C6, R1, R10, R11, R12, R13, R14, R15, R16, R17, R18, R19, R2, R20, R21, R22, R23, R24, R25, R26, R27, R28, R29, R3, R30, R31, R32, R33, R34, R35, R36, R37, R38, R39, R4, R5, R6, R7, R8, R9: footprint carbon_hero:0402 -> patamana:0402
- J1, J2: footprint carbon_hero:MJ-4PP-9 -> patamana:MJ-4PP-9
- SW1, SW2: footprint carbon_hero:Tactile_Switch_TVDP01 -> patamana:Tactile_Switch_TVDP01
- SW3, SW4: footprint carbon_hero:SS-12D00-G5 -> patamana:SS-12D00-G5
- U1: footprint carbon_hero:XIAO_ESP32S3 -> patamana:XIAO_ESP32S3
- U2, U4, U5, U6: footprint carbon_hero:SOT109-1_SO16 -> patamana:SOT109-1_SO16
- U3: footprint carbon_hero:OLED_128x64_I2C -> patamana:OLED_128x64_I2C
- U7: footprint carbon_hero:patamana_0_4_out -> patamana:patamana_0_4_out
