File: kicad/patamana.kicad_sch (KiCad schematic)
At the start: 59 parts, among them J1 TRRSJack, J2 Conn_01x02, SW2 SW_Push, SW3 SW_DPDT_x2, SW4 SW_DPDT_x2, SW4 SW_Push, U1 XIAO_ESP32S3, U2 OLED(I2C), U3 74HC165, U4 74HC165, U5 74HC165, U6 74HC165

Commit message: 整理:名前の整理
Parts:
- C1, C2, C3, C4, C5, C6, R1, R10, R11, R12, R13, R14, R15, R16, R17, R18, R19, R2, R20, R21, R22, R23, R24, R25, R26, R27, R28, R29, R3, R30, R31, R32, R33, R34, R35, R36, R37, R38, R39, R4, R40, R5, R7, R8, R9: footprint carbon_hero:0402 -> patamana:0402
- J1: footprint carbon_hero:MJ-4PP-9 -> patamana:MJ-4PP-9
- SW2, SW4: footprint carbon_hero:Tactile_Switch_TVDP01 -> patamana:Tactile_Switch_TVDP01
- SW3, SW4: footprint carbon_hero:SS-12D00-G5 -> patamana:SS-12D00-G5
- U1: footprint carbon_hero:XIAO_ESP32S3 -> patamana:XIAO_ESP32S3; symbol carbon_hero:XIAO_ESP32S3 -> patamana:XIAO_ESP32S3
- U2: footprint carbon_hero:OLED_128x64_I2C -> patamana:OLED_128x64_I2C; symbol carbon_hero:I2C -> patamana:I2C
- U3, U4, U5, U6: footprint carbon_hero:SOT109-1_SO16 -> patamana:SOT109-1_SO16; symbol carbon_hero:74hc165 -> patamana:74hc165
- U7: footprint carbon_hero:patamana_0_4_out -> patamana:patamana_0_4_out; symbol carbon_hero:patamana_out -> patamana:patamana_out
